Commit message: [pcd_filter et al] Rename the preprocessing package to pcd_filter and standardize filtering topics and node names

File: aerial_motion/pcd_filter/test/robot.urdf (robot description, URDF)
Before this commit: robot self_filter_test, 4 links, 3 joints
Links:
- link mesh: geometry collision mesh filename=package://pcd_filter/test/tetrahedron.stl scale=0.5 0.5 0.5
